Commit message: Added camera sensor to robot on URDF.

File: ros_intro/go_chase_it_project/catkin_ws/src/my_robot/urdf/my_robot.xacro (robot description, xacro)
@@ -7,4 +7,56 @@
     <child link="chassis" />
   </joint>
+  <!-- CHASSIS -->
+  <link name='chassis'>
+    <pose>0 0 0.1 0 0 0</pose>
+    <inertial>
+      <mass value="15.0"/>
+      <origin xyz="0.0 0 0" rpy=" 0 0 0"/>
+      <inertia
+          ixx="0.1" ixy="0" ixz="0"
+          iyy="0.1" iyz="0"
+          izz="0.1"
+      />
+    </inertial>
+    <collision name='collision'>
+      <origin xyz="0 0 0" rpy=" 0 0 0"/>
+      <geometry>
+        <box size=".4 .2 .1"/>
+      </geometry>
+    </collision>
+    <visual name='chassis_visual'>
+      <origin xyz="0 0 0" rpy=" 0 0 0"/>
+      <geometry>
+        <box size=".4 .2 .1"/>
+      </geometry>
+    </visual>
+    <!-- BACK CASTER -->
+    <collision name='back_caster_collision'>
+      <origin xyz="-0.15 0 -0.05" rpy=" 0 0 0"/>
+      <geometry>
+        <sphere radius="0.0499"/>
+      </geometry>
+    </collision>
+    <visual name='back_caster_visual'>
+      <origin xyz="-0.15 0 -0.05" rpy=" 0 0 0"/>
+      <geometry>
+        <sphere radius="0.05"/>
+      </geometry>
+    </visual>
+    <!-- FRONT CASTER -->
+    <collision name='front_caster_collision'>
+      <origin xyz="0.15 0 -0.05" rpy=" 0 0 0"/>
+      <geometry>
+        <sphere radius="0.0499"/>
+      </geometry>
+    </collision>
+    <visual name='front_caster_visual'>
+      <origin xyz="0.15 0 -0.05" rpy=" 0 0 0"/>
+      <geometry>
+        <sphere radius="0.05"/>
+      </geometry>
+    </visual>
+  </link>
+  <!-- LEFT WHEEL -->
   <link name="left_wheel">
     <pose>0 0 0 0 0 0</pose>
@@ -39,4 +91,5 @@
     <dynamics damping="1.0" friction="1.0"/>
   </joint>
+  <!-- RIGHT WHEEL -->
   <link name="right_wheel">
     <pose>0 0 0 0 0 0</pose>
@@ -71,51 +124,36 @@
     <dynamics damping="1.0" friction="1.0"/>
   </joint>
-  <link name='chassis'>
-    <pose>0 0 0.1 0 0 0</pose>
+  <!-- CAMERA -->
+  <link name="camera">
+    <pose>0 0 0 0 0 0</pose>
     <inertial>
-      <mass value="15.0"/>
-      <origin xyz="0.0 0 0" rpy=" 0 0 0"/>
+      <mass value="0.1"/>
+      <origin xyz="0.0 0 0" rpy=" 0, 0, 0"/>
       <inertia
-          ixx="0.1" ixy="0" ixz="0"
-          iyy="0.1" iyz="0"
-          izz="0.1"
+          ixx="1e-6" ixy="0" ixz="0"
+          iyy="1e-6" iyz="0"
+          izz="1e-6"
       />
     </inertial>
-    <collision name='collision'>
-      <origin xyz="0 0 0" rpy=" 0 0 0"/>
+    <collision name='camera_collision'>
+      <origin xyz="0 0 0" rpy=" 0, 0, 0"/>
       <geometry>
-        <box size=".4 .2 .1"/>
+        <box size="0.05 0.05 0.05" />
       </geometry>
     </collision>
-    <visual name='chassis_visual'>
-      <origin xyz="0 0 0" rpy=" 0 0 0"/>
+    <visual name='camera_visual'>
+      <origin xyz="0 0 0" rpy=" 0, 0, 0"/>
       <geometry>
-        <box size=".4 .2 .1"/>
-      </geometry>
-    </visual>
-    <collision name='back_caster_collision'>
-      <origin xyz="-0.15 0 -0.05" rpy=" 0 0 0"/>
-      <geometry>
-        <sphere radius="0.0499"/>
-      </geometry>
-    </collision>
-    <visual name='back_caster_visual'>
-      <origin xyz="-0.15 0 -0.05" rpy=" 0 0 0"/>
-      <geometry>
-        <sphere radius="0.05"/>
-      </geometry>
-    </visual>
-    <collision name='front_caster_collision'>
-      <origin xyz="0.15 0 -0.05" rpy=" 0 0 0"/>
-      <geometry>
-        <sphere radius="0.0499"/>
-      </geometry>
-    </collision>
-    <visual name='front_caster_visual'>
-      <origin xyz="0.15 0 -0.05" rpy=" 0 0 0"/>
-      <geometry>
-        <sphere radius="0.05"/>
+        <box size="0.05 0.05 0.05" />
       </geometry>
     </visual>
   </link>
+  <joint type="fixed" name="camera_joint">
+    <origin xyz="0.2 0 0" rpy="0 0 0"/>
+    <child link="camera"/>
+    <parent link="chassis"/>
+    <axis xyz="0 1 0" rpy="0 0 0"/>
+    <limit effort="10000" velocity="1000"/>
+    <dynamics damping="1.0" friction="1.0"/>
+  </joint>
 </robot>

Commit message: Added both lidar and camera onto robot. Added colors via materials in URDF.

File: ros_intro/go_chase_it_project/catkin_ws/src/my_robot/urdf/my_robot.xacro (robot description, xacro)
@@ -1,4 +1,17 @@
 <?xml version='1.0'?>
 <robot name="my_robot" xmlns:xacro="http://www.ros.org/wiki/xacro">
+  <!-- COLORS -->
+  <gazebo reference="left_wheel">
+    <material>Gazebo/Gray</material>
+  </gazebo>
+  <gazebo reference="right_wheel">
+    <material>Gazebo/Gray</material>
+  </gazebo>
+  <gazebo reference="chassis">
+    <material>Gazebo/Red</material>
+  </gazebo>
+  <gazebo reference="camera">
+    <material>Gazebo/Blue</material>
+  </gazebo>
   <link name="robot_footprint"></link>
   <joint name="robot_footprint_joint" type="fixed">
@@ -157,3 +170,36 @@
     <dynamics damping="1.0" friction="1.0"/>
   </joint>
+  <!-- LIDAR -->
+  <link name="hokuyo">
+    <pose>0 0 0 0 0 0</pose>
+    <inertial>
+      <mass value="1e-5"/>
+      <origin xyz="0.0 0 0" rpy=" 0, 0, 0"/>
+      <inertia
+          ixx="1e-6" ixy="0" ixz="0"
+          iyy="1e-6" iyz="0"
+          izz="1e-6"
+      />
+    </inertial>
+    <collision name='hokuyo_collision'>
+      <origin xyz="0 0 0" rpy=" 0, 0, 0"/>
+      <geometry>
+        <box size="0.1 0.1 0.1" />
+      </geometry>
+    </collision>
+    <visual name='hokuyo_visual'>
+      <origin xyz="0 0 0" rpy=" 0, 0, 0"/>
+      <geometry>
+        <mesh filename="package://my_robot/meshes/hokuyo.dae"/>
+      </geometry>
+    </visual>
+  </link>
+  <joint type="fixed" name="hokuyo_joint">
+    <origin xyz="0.15 0 0.1" rpy="0 0 0"/>
+    <child link="hokuyo"/>
+    <parent link="chassis"/>
+    <axis xyz="0 1 0" rpy="0 0 0"/>
+    <limit effort="10000" velocity="1000"/>
+    <dynamics damping="1.0" friction="1.0"/>
+  </joint>
 </robot>

Commit message: Added code to integrate RViz with Gazebo. Now, whatever sensors mounted on robot (lidar and camera) perceives are published in topics, and can be subscribed in RViz for visualization purposes.

File: ros_intro/go_chase_it_project/catkin_ws/src/my_robot/urdf/my_robot.xacro (robot description, xacro)
@@ -1,4 +1,6 @@
 <?xml version='1.0'?>
 <robot name="my_robot" xmlns:xacro="http://www.ros.org/wiki/xacro">
+  <!-- PLUGINS FOR ROBOT -->
+  <xacro:include filename="$(find my_robot)/urdf/my_robot.gazebo" />
   <!-- COLORS -->
   <gazebo reference="left_wheel">
@@ -76,5 +78,5 @@
     <inertial>
       <mass value="5.0"/>
-      <origin xyz="0.0 0 0" rpy=" 0, 1.5707, 1.5707"/>
+      <origin xyz="0.0 0 0" rpy=" 0 1.5707 1.5707"/>
       <inertia
           ixx="0.1" ixy="0" ixz="0"
@@ -84,5 +86,5 @@
     </inertial>
     <collision name='left_wheel_collision'>
-      <origin xyz="0 0 0" rpy=" 0, 1.5707, 1.5707"/>
+      <origin xyz="0 0 0" rpy=" 0 1.5707 1.5707"/>
       <geometry>
         <cylinder length="0.05" radius="0.1"/>
@@ -90,5 +92,5 @@
     </collision>
     <visual name='left_wheel_visual'>
-      <origin xyz="0 0 0" rpy=" 0, 1.5707, 1.5707"/>
+      <origin xyz="0 0 0" rpy=" 0 1.5707 1.5707"/>
       <geometry>
         <cylinder length="0.05" radius="0.1"/>
@@ -109,5 +111,5 @@
     <inertial>
       <mass value="5.0"/>
-      <origin xyz="0.0 0 0" rpy=" 0, 1.5707, 1.5707"/>
+      <origin xyz="0.0 0 0" rpy=" 0 1.5707 1.5707"/>
       <inertia
           ixx="0.1" ixy="0" ixz="0"
@@ -117,5 +119,5 @@
     </inertial>
     <collision name='right_wheel_collision'>
-      <origin xyz="0 0 0" rpy=" 0, 1.5707, 1.5707"/>
+      <origin xyz="0 0 0" rpy=" 0 1.5707 1.5707"/>
       <geometry>
         <cylinder length="0.05" radius="0.1"/>
@@ -123,5 +125,5 @@
     </collision>
     <visual name='right_wheel_visual'>
-      <origin xyz="0 0 0" rpy=" 0, 1.5707, 1.5707"/>
+      <origin xyz="0 0 0" rpy=" 0 1.5707 1.5707"/>
       <geometry>
         <cylinder length="0.05" radius="0.1"/>
@@ -142,5 +144,5 @@
     <inertial>
       <mass value="0.1"/>
-      <origin xyz="0.0 0 0" rpy=" 0, 0, 0"/>
+      <origin xyz="0.0 0 0" rpy=" 0 0 0"/>
       <inertia
           ixx="1e-6" ixy="0" ixz="0"
@@ -150,5 +152,5 @@
     </inertial>
     <collision name='camera_collision'>
-      <origin xyz="0 0 0" rpy=" 0, 0, 0"/>
+      <origin xyz="0 0 0" rpy=" 0 0 0"/>
       <geometry>
         <box size="0.05 0.05 0.05" />
@@ -156,5 +158,5 @@
     </collision>
     <visual name='camera_visual'>
-      <origin xyz="0 0 0" rpy=" 0, 0, 0"/>
+      <origin xyz="0 0 0" rpy=" 0 0 0"/>
       <geometry>
         <box size="0.05 0.05 0.05" />
@@ -175,5 +177,5 @@
     <inertial>
       <mass value="1e-5"/>
-      <origin xyz="0.0 0 0" rpy=" 0, 0, 0"/>
+      <origin xyz="0.0 0 0" rpy=" 0 0 0"/>
       <inertia
           ixx="1e-6" ixy="0" ixz="0"
@@ -183,5 +185,5 @@
     </inertial>
     <collision name='hokuyo_collision'>
-      <origin xyz="0 0 0" rpy=" 0, 0, 0"/>
+      <origin xyz="0 0 0" rpy=" 0 0 0"/>
       <geometry>
         <box size="0.1 0.1 0.1" />
@@ -189,5 +191,5 @@
     </collision>
     <visual name='hokuyo_visual'>
-      <origin xyz="0 0 0" rpy=" 0, 0, 0"/>
+      <origin xyz="0 0 0" rpy=" 0 0 0"/>
       <geometry>
         <mesh filename="package://my_robot/meshes/hokuyo.dae"/>
