Commit message: Converted 2D Camera to 3D camera - kinect sensor.

File: projects/rtab_map_slam_project/catkin_ws/src/my_robot/urdf/my_robot.xacro (robot description, xacro)
@@ -16,4 +16,13 @@
     <material>Gazebo/Blue</material>
   </gazebo>
+  <!-- 3D CAMERA DEPTH SENSOR JOINT -->
+  <joint name="camera_optical_joint" type="fixed">
+    <origin xyz="0 0 0" rpy="-1.5707 0 -1.5707"/>
+    <parent link="camera"/>
+    <child link="camera_link_optical"/>
+  </joint>
+  <link name="camera_link_optical">
+  </link>
+  <!-- ROBOT FOOTPRINT -->
   <link name="robot_footprint"></link>
   <joint name="robot_footprint_joint" type="fixed">
