Commit message: Adjusted parameters for AMCL to work better.

File: projects/monte_carlo_localization_project/catkin_ws/src/my_robot/urdf/my_robot.xacro (robot description, xacro)
@@ -11,8 +11,8 @@
   </gazebo>
   <gazebo reference="chassis">
-    <material>Gazebo/Red</material>
+    <material>Gazebo/Blue</material>
   </gazebo>
   <gazebo reference="camera">
-    <material>Gazebo/Blue</material>
+    <material>Gazebo/Green</material>
   </gazebo>
   <link name="robot_footprint"></link>
